File: KiCad_PCB_Files/Version 2.2/Arduino_Board_Only_Spot_Welder.kicad_pcb (KiCad board)
At the start: 2 copper layers, 50 x 60 mm, 35 parts, among them P1 MCP1407, P2 GND_con, P3 GND_con, U1 arduino_nano

Commit message: Add files via upload
Parts:
- removed R13: 20k, Resistors_SMD:R_1206_HandSoldering
- R15: value 470 -> 620
Routing:
- net /D3: track 37.3 -> 33.3 mm
- net GND: track 60.8 -> 59.5 mm
