File: KiCad_PCB_Files/Version 2.2/Arduino_Spot_Welder.kicad_pcb (KiCad board)
At the start: 2 copper layers, 110 x 60 mm, 58 parts, among them P1 MCP1407, P2 GND_con, P3 GND_con, P4 GND_con, P5 GND_con, Q1 IRF1405, Q2 IRF1405, Q3 IRF1405, Q4 IRF1405, Q5 IRF1405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

Commit message: Add files via upload
Parts:
- removed R13: 20k, Resistors_SMD:R_1206_HandSoldering
- Q1, Q2, Q3, Q4, Q5, Q6, Q7, Q8: value IRF1405 -> IRFB_7437
- R15: value 470 -> 620
Routing:
- net /D3: track 37.3 -> 33.3 mm
- net GND: track 60.8 -> 59.5 mm
Changed lines of the file:
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@@
 (kicad_pcb (version 4) (host pcbnew 4.0.4-stable)
   (general
-    (links 91)
+    (links 89)
     (no_connects 8)
     (area 69.924999 69.924999 180.075001 130.075001)
     (thickness 1.6)
-    (drawings 48)
-    (tracks 387)
+    (drawings 52)
+    (tracks 380)
     (zones 0)
-    (modules 58)
+    (modules 57)
     (nets 55)
   )
@@
     (40 Dwgs.User user hide)
     (41 Cmts.User user)
-    (42 Eco1.User user hide)
+    (42 Eco1.User user)
     (43 Eco2.User user hide)
     (44 Edge.Cuts user)
@@
   )
   (setup
-    (last_trace_width 0.35)
+    (last_trace_width 0.25)
     (user_trace_width 0.35)
     (user_trace_width 0.5)
@@
       (effects (font (size 1 1) (thickness 0.15)))
     )
-    (fp_text value IRF1405 (at -4 -8 360) (layer F.SilkS)
+    (fp_text value IRFB_7437 (at -3 -8 360) (layer F.SilkS)
       (effects (font (size 1 1) (thickness 0.15)))
     )
@@
       (effects (font (size 1 1) (thickness 0.15)))
     )
-    (fp_text value IRF1405 (at 4 -7.5 180) (layer F.SilkS)
+    (fp_text value IRFB_7437 (at 3 -8 180) (layer F.SilkS)
       (effects (font (size 1 1) (thickness 0.15)))
     )
@@
       (effects (font (size 1 1) (thickness 0.15)))
     )
-    (fp_text value IRF1405 (at 4 -7.5 180) (layer F.SilkS)
+    (fp_text value IRFB_7437 (at 3 -8 180) (layer F.SilkS)
       (effects (font (size 1 1) (thickness 0.15)))
     )
@@
       (effects (font (size 1 1) (thickness 0.15)))
     )
-    (fp_text value IRF1405 (at 4 -7.5 180) (layer F.SilkS)
+    (fp_text value IRFB_7437 (at 3 -8 180) (layer F.SilkS)
       (effects (font (size 1 1) (thickness 0.15)))
     )
@@
       (effects (font (size 1 1) (thickness 0.15)))
     )
-    (fp_text value IRF1405 (at 4 -7.5 180) (layer F.SilkS)
+    (fp_text value IRFB_7437 (at 3 -8 180) (layer F.SilkS)
       (effects (font (size 1 1) (thickness 0.15)))
     )
@@
       (effects (font (size 1 1) (thickness 0.15)))
     )
-    (fp_text value IRF1405 (at -4 -8 360) (layer F.SilkS)
+    (fp_text value IRFB_7437 (at -3 -8 360) (layer F.SilkS)
       (effects (font (size 1 1) (thickness 0.15)))
     )
@@
       (effects (font (size 1 1) (thickness 0.15)))
     )
-    (fp_text value IRF1405 (at -4 -8 360) (layer F.SilkS)
+    (fp_text value IRFB_7437 (at -3 -8 360) (layer F.SilkS)
       (effects (font (size 1 1) (thickness 0.15)))
     )
@@
       (effects (font (size 1 1) (thickness 0.15)))
     )
-    (fp_text value IRF1405 (at -4 -8 360) (layer F.SilkS)
+    (fp_text value IRFB_7437 (at -3 -8 360) (layer F.SilkS)
       (effects (font (size 1 1) (thickness 0.15)))
     )
@@
   )
   (module Resistors_SMD:R_1206_HandSoldering (layer F.Cu)
-    (at 91.75 81.75)
-    (descr "Resistor SMD 1206, hand soldering")
-    (tags "resistor 1206")
-    (attr smd)
-    (fp_text reference R13 (at -2 -1.75) (layer F.SilkS)
-      (effects (font (size 1 1) (thickness 0.15)))
-    )
-    (fp_text value 20k (at 1.75 -1.75) (layer F.SilkS)
-      (effects (font (size 1 1) (thickness 0.15)))
-    )
-    (fp_text user %R (at 0 0) (layer F.Fab)
-      (effects (font (size 0.7 0.7) (thickness 0.105)))
-    )
-    (fp_line (start -1.6 0.8) (end -1.6 -0.8) (layer F.Fab) (width 0.1))
-    (fp_line (start 1.6 0.8) (end -1.6 0.8) (layer F.Fab) (width 0.1))
-    (fp_line (start 1.6 -0.8) (end 1.6 0.8) (layer F.Fab) (width 0.1))
-    (fp_line (start -1.6 -0.8) (end 1.6 -0.8) (layer F.Fab) (width 0.1))
-    (fp_line (start 1 1.07) (end -1 1.07) (layer F.SilkS) (width 0.12))
-    (fp_line (start -1 -1.07) (end 1 -1.07) (layer F.SilkS) (width 0.12))
-    (fp_line (start -3.25 -1.11) (end 3.25 -1.11) (layer F.CrtYd) (width 0.05))
-    (fp_line (start -3.25 -1.11) (end -3.25 1.1) (layer F.CrtYd) (width 0.05))
-    (fp_line (start 3.25 1.1) (end 3.25 -1.11) (layer F.CrtYd) (width 0.05))
-    (fp_line (start 3.25 1.1) (end -3.25 1.1) (layer F.CrtYd) (width 0.05))
-    (pad 1 smd rect (at -2 0) (size 2 1.7) (layers F.Cu F.Paste F.Mask)
-      (net 54 /D3))
-    (pad 2 smd rect (at 2 0) (size 2 1.7) (layers F.Cu F.Paste F.Mask)
-      (net 2 GND))
-    (model ${KISYS3DMOD}/Resistors_SMD.3dshapes/R_1206.wrl
-      (at (xyz 0 0 0))
-      (scale (xyz 1 1 1))
-      (rotate (xyz 0 0 0))
-    )
-  )
-  (module Resistors_SMD:R_1206_HandSoldering (layer F.Cu)
     (at 83.75 81.75)
     (descr "Resistor SMD 1206, hand soldering")
@@
       (effects (font (size 1 1) (thickness 0.15)))
     )
-    (fp_text value 470 (at -1.25 -2 180) (layer F.SilkS)
+    (fp_text value 620 (at -1.25 -2 180) (layer F.SilkS)
       (effects (font (size 1 1) (thickness 0.15)))
     )
@@
       (rotate (xyz 0 0 0))
     )
+  )
+  (dimension 60 (width 0.3) (layer Eco1.User)
+    (gr_text "60.000 mm" (at 186.35 100 270) (layer Eco1.User)
+      (effects (font (size 1.5 1.5) (thickness 0.3)))
+    )
+    (feature1 (pts (xy 180 130) (xy 187.7 130)))
+    (feature2 (pts (xy 180 70) (xy 187.7 70)))
+    (crossbar (pts (xy 185 70) (xy 185 130)))
+    (arrow1a (pts (xy 185 130) (xy 184.413579 128.873496)))
+    (arrow1b (pts (xy 185 130) (xy 185.586421 128.873496)))
+    (arrow2a (pts (xy 185 70) (xy 184.413579 71.126504)))
+    (arrow2b (pts (xy 185 70) (xy 185.586421 71.126504)))
+  )
+  (dimension 50 (width 0.3) (layer Eco1.User)
+    (gr_text "50.000 mm" (at 155 62.65) (layer Eco1.User)
+      (effects (font (size 1.5 1.5) (thickness 0.3)))
+    )
+    (feature1 (pts (xy 180 70) (xy 180 61.3)))
+    (feature2 (pts (xy 130 70) (xy 130 61.3)))
+    (crossbar (pts (xy 130 64) (xy 180 64)))
+    (arrow1a (pts (xy 180 64) (xy 178.873496 64.586421)))
+    (arrow1b (pts (xy 180 64) (xy 178.873496 63.413579)))
+    (arrow2a (pts (xy 130 64) (xy 131.126504 64.586421)))
+    (arrow2b (pts (xy 130 64) (xy 131.126504 63.413579)))
+  )
+  (dimension 60 (width 0.3) (layer Eco1.User)
+    (gr_text "60.000 mm" (at 63.650001 100 270) (layer Eco1.User)
+      (effects (font (size 1.5 1.5) (thickness 0.3)))
+    )
+    (feature1 (pts (xy 70 130) (xy 62.300001 130)))
+    (feature2 (pts (xy 70 70) (xy 62.300001 70)))
+    (crossbar (pts (xy 65.000001 70) (xy 65.000001 130)))
+    (arrow1a (pts (xy 65.000001 130) (xy 64.41358 128.873496)))
+    (arrow1b (pts (xy 65.000001 130) (xy 65.586422 128.873496)))
+    (arrow2a (pts (xy 65.000001 70) (xy 64.41358 71.126504)))
+    (arrow2b (pts (xy 65.000001 70) (xy 65.586422 71.126504)))
+  )
+  (dimension 50 (width 0.3) (layer Eco1.User)
+    (gr_text "50.000 mm" (at 95 62.65) (layer Eco1.User)
+      (effects (font (size 1.5 1.5) (thickness 0.3)))
+    )
+    (feature1 (pts (xy 120 70) (xy 120 61.3)))
+    (feature2 (pts (xy 70 70) (xy 70 61.3)))
+    (crossbar (pts (xy 70 64) (xy 120 64)))
+    (arrow1a (pts (xy 120 64) (xy 118.873496 64.586421)))
+    (arrow1b (pts (xy 120 64) (xy 118.873496 63.413579)))
+    (arrow2a (pts (xy 70 64) (xy 71.126504 64.586421)))
+    (arrow2b (pts (xy 70 64) (xy 71.126504 63.413579)))
   )
   (gr_line (start 101.7 82.75) (end 101.7 83.3) (angle 90) (layer F.SilkS) (width 0.1))
@@
   (segment (start 73.5 79.37) (end 76.49 76.38) (width 0.5) (layer F.Cu) (net 1))
   (segment (start 73.5 97) (end 73.5 79.37) (width 0.5) (layer F.Cu) (net 1))
-  (segment (start 93.75 81.75) (end 95.25 81.75) (width 0.35) (layer F.Cu) (net 2))
-  (segment (start 96.25 82.75) (end 98.75 82.75) (width 0.35) (layer F.Cu) (net 2))
-  (segment (start 95.25 81.75) (end 96.25 82.75) (width 0.35) (layer F.Cu) (net 2))
+  (segment (start 98.75 82.75) (end 89.25 82.75) (width 0.35) (layer F.Cu) (net 2))
+  (segment (start 89 83) (end 89 86) (width 0.35) (layer F.Cu) (net 2))
+  (segment (start 89.25 82.75) (end 89 83) (width 0.35) (layer F.Cu) (net 2))
   (segment (start 87.25 72) (end 82.54 72) (width 0.35) (layer F.Cu) (net 2))
-  (segment (start 89 83.75) (end 89 86) (width 0.35) (layer F.Cu) (net 2))
-  (segment (start 89.25 83.5) (end 89 83.75) (width 0.35) (layer F.Cu) (net 2))
-  (segment (start 89.75 83.5) (end 89.25 83.5) (width 0.35) (layer F.Cu) (net 2))
-  (segment (start 93.5 83.5) (end 89.75 83.5) (width 0.35) (layer F.Cu) (net 2))
-  (segment (start 93.75 83.25) (end 93.5 83.5) (width 0.35) (layer F.Cu) (net 2))
-  (segment (start 93.75 81.75) (end 93.75 83.25) (width 0.35) (layer F.Cu) (net 2))
   (segment (start 76.4 104.3) (end 76.7 104.3) (width 1) (layer B.Cu) (net 2))
   (segment (start 76.7 104.3) (end 76.65 104.25) (width 1) (layer F.Cu) (net 2))
@@
   (segment (start 85.75 84.5) (end 86.25 85) (width 0.35) (layer F.Cu) (net 54))
   (segment (start 85.75 81.75) (end 85.75 84.5) (width 0.35) (layer F.Cu) (net 54))
-  (segment (start 85.75 81.75) (end 89.75 81.75) (width 0.35) (layer F.Cu) (net 54))
   (zone (net 2) (net_name GND) (layer B.Cu) (hatch edge 0.508)
     (connect_pads (clearance 0.508))
