File: KiCad_PCB_Files/Version 2.2/Arduino_Spot_Welder.sch (KiCad schematic (older format))
At the start: 42 parts, among them P1 MCP1407, P2 GND_con, P3 GND_con, P4 GND_con, P5 GND_con, Q1 IRF1405, Q2 IRF1405, Q3 IRF1405, Q4 IRF1405, Q5 IRF1405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

Commit message: Add files via upload
Parts:
- removed R13: 20k, Resistors_SMD:R_1206_HandSoldering, symbol R
- Q1, Q2, Q3, Q4, Q5, Q6, Q7, Q8: value IRF1405 -> IRFB_7437
- R15: value 470 -> 620
Other:
- moved on the sheet: D3
Changed lines of the file:
@@
 P 7000 3050
 F 0 "Q2" H 7250 3125 50  0000 L CNN
-F 1 "IRF1405" H 7250 3050 50  0000 L CNN
+F 1 "IRFB_7437" H 7250 3050 50  0000 L CNN
 F 2 "pots_own:TO-220__long_Neutral123_Horizontal_LargePads" H 7250 2975 50  0001 L CIN
 F 3 "" H 7000 3050 50  0000 L CNN
@@
 P 7625 3050
 F 0 "Q3" H 7875 3125 50  0000 L CNN
-F 1 "IRF1405" H 7875 3050 50  0000 L CNN
+F 1 "IRFB_7437" H 7875 3050 50  0000 L CNN
 F 2 "pots_own:TO-220__long_Neutral123_Horizontal_LargePads" H 7875 2975 50  0001 L CIN
 F 3 "" H 7625 3050 50  0000 L CNN
@@
 P 8200 3050
 F 0 "Q4" H 8450 3125 50  0000 L CNN
-F 1 "IRF1405" H 8450 3050 50  0000 L CNN
+F 1 "IRFB_7437" H 8450 3050 50  0000 L CNN
 F 2 "pots_own:TO-220__long_Neutral123_Horizontal_LargePads" H 8450 2975 50  0001 L CIN
 F 3 "" H 8200 3050 50  0000 L CNN
@@
 P 8800 3050
 F 0 "Q5" H 9050 3125 50  0000 L CNN
-F 1 "IRF1405" H 9050 3050 50  0000 L CNN
+F 1 "IRFB_7437" H 9050 3050 50  0000 L CNN
 F 2 "pots_own:TO-220__long_Neutral123_Horizontal_LargePads" H 9050 2975 50  0001 L CIN
 F 3 "" H 8800 3050 50  0000 L CNN
@@
 P 9375 3050
 F 0 "Q6" H 9625 3125 50  0000 L CNN
-F 1 "IRF1405" H 9625 3050 50  0000 L CNN
+F 1 "IRFB_7437" H 9625 3050 50  0000 L CNN
 F 2 "pots_own:TO-220__long_Neutral123_Horizontal_LargePads" H 9625 2975 50  0001 L CIN
 F 3 "" H 9375 3050 50  0000 L CNN
@@
 P 9950 3050
 F 0 "Q7" H 10200 3125 50  0000 L CNN
-F 1 "IRF1405" H 10200 3050 50  0000 L CNN
+F 1 "IRFB_7437" H 10200 3050 50  0000 L CNN
 F 2 "pots_own:TO-220__long_Neutral123_Horizontal_LargePads" H 10200 2975 50  0001 L CIN
 F 3 "" H 9950 3050 50  0000 L CNN
@@
 P 10575 3050
 F 0 "Q8" H 10825 3125 50  0000 L CNN
-F 1 "IRF1405" H 10825 3050 50  0000 L CNN
+F 1 "IRFB_7437" H 10825 3050 50  0000 L CNN
 F 2 "pots_own:TO-220__long_Neutral123_Horizontal_LargePads" H 10825 2975 50  0001 L CIN
 F 3 "" H 10575 3050 50  0000 L CNN
@@
 P 6400 3050
 F 0 "Q1" H 6650 3125 50  0000 L CNN
-F 1 "IRF1405" H 6650 3050 50  0000 L CNN
+F 1 "IRFB_7437" H 6650 3050 50  0000 L CNN
 F 2 "pots_own:TO-220__long_Neutral123_Horizontal_LargePads" H 6650 2975 50  0001 L CIN
 F 3 "" H 6400 3050 50  0000 L CNN
@@
 D3
 $Comp
-L R R13
-U 1 1 5904FD0C
-P 3800 4950
-F 0 "R13" V 3880 4950 50  0000 C CNN
-F 1 "20k" V 3800 4950 50  0000 C CNN
-F 2 "Resistors_SMD:R_1206_HandSoldering" V 3730 4950 50  0001 C CNN
-F 3 "" H 3800 4950 50  0000 C CNN
-	1    3800 4950
-	0    1    1    0
-$EndComp
-$Comp
 L R R14
 U 1 1 5904FF40
@@
 P 4225 4450
 F 0 "R15" V 4305 4450 50  0000 C CNN
-F 1 "470" V 4225 4450 50  0000 C CNN
+F 1 "620" V 4225 4450 50  0000 C CNN
 F 2 "Resistors_SMD:R_1206_HandSoldering" V 4155 4450 50  0001 C CNN
 F 3 "" H 4225 4450 50  0000 C CNN
@@
 Connection ~ 6800 2300
 Wire Wire Line
-	3475 4950 3650 4950
-Wire Wire Line
 	4075 4950 3950 4950
 Wire Wire Line
@@
 L ZENER D3
 U 1 1 5907549C
-P 3700 4750
-F 0 "D3" H 3700 4850 50  0000 C CNN
-F 1 "ZENER" H 3700 4650 50  0000 C CNN
-F 2 "Diodes_SMD:D_MiniMELF_Handsoldering" H 3700 4750 50  0001 C CNN
-F 3 "" H 3700 4750 50  0000 C CNN
-	1    3700 4750
+P 3750 4950
+F 0 "D3" H 3750 5050 50  0000 C CNN
+F 1 "ZENER" H 3750 4850 50  0000 C CNN
+F 2 "Diodes_SMD:D_MiniMELF_Handsoldering" H 3750 4950 50  0001 C CNN
+F 3 "" H 3750 4950 50  0000 C CNN
+	1    3750 4950
 	-1   0    0    1
 $EndComp
-Wire Wire Line
-	3900 4750 4000 4750
-Connection ~ 4000 4750
-Wire Wire Line
-	3500 4950 3500 4750
 Connection ~ 3500 4950
+Wire Wire Line
+	3475 4950 3550 4950
 $EndSCHEMATC
