File: KiCad_PCB_Files/Version 2.2/Mosfet_Board_Only_Spot_Welder.kicad_pcb (KiCad board)
At the start: 2 copper layers, 50 x 60 mm, 23 parts, among them P4 GND_con, P5 GND_con, Q1 IRF1405, Q2 IRF1405, Q3 IRF1405, Q4 IRF1405, Q5 IRF1405, Q6 IRF1405, Q7 IRF1405, Q8 IRF1405

Commit message: Add files via upload
Parts:
- Q1, Q2, Q3, Q4, Q5, Q6, Q7, Q8: value IRF1405 -> IRFB_7437
Changed lines of the file:
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@@
       (effects (font (size 1 1) (thickness 0.15)))
     )
-    (fp_text value IRF1405 (at -4 -8 360) (layer F.SilkS)
+    (fp_text value IRFB_7437 (at -3 -8 360) (layer F.SilkS)
       (effects (font (size 1 1) (thickness 0.15)))
     )
@@
       (effects (font (size 1 1) (thickness 0.15)))
     )
-    (fp_text value IRF1405 (at 4 -7.5 180) (layer F.SilkS)
+    (fp_text value IRFB_7437 (at 3 -8 180) (layer F.SilkS)
       (effects (font (size 1 1) (thickness 0.15)))
     )
@@
       (effects (font (size 1 1) (thickness 0.15)))
     )
-    (fp_text value IRF1405 (at 4 -7.5 180) (layer F.SilkS)
+    (fp_text value IRFB_7437 (at 3 -8 180) (layer F.SilkS)
       (effects (font (size 1 1) (thickness 0.15)))
     )
@@
       (effects (font (size 1 1) (thickness 0.15)))
     )
-    (fp_text value IRF1405 (at 4 -7.5 180) (layer F.SilkS)
+    (fp_text value IRFB_7437 (at 3 -8 180) (layer F.SilkS)
       (effects (font (size 1 1) (thickness 0.15)))
     )
@@
       (effects (font (size 1 1) (thickness 0.15)))
     )
-    (fp_text value IRF1405 (at 4 -7.5 180) (layer F.SilkS)
+    (fp_text value IRFB_7437 (at 3 -8 180) (layer F.SilkS)
       (effects (font (size 1 1) (thickness 0.15)))
     )
@@
       (effects (font (size 1 1) (thickness 0.15)))
     )
-    (fp_text value IRF1405 (at -4 -8 360) (layer F.SilkS)
+    (fp_text value IRFB_7437 (at -3 -8 360) (layer F.SilkS)
       (effects (font (size 1 1) (thickness 0.15)))
     )
@@
       (effects (font (size 1 1) (thickness 0.15)))
     )
-    (fp_text value IRF1405 (at -4 -8 360) (layer F.SilkS)
+    (fp_text value IRFB_7437 (at -3 -8 360) (layer F.SilkS)
       (effects (font (size 1 1) (thickness 0.15)))
     )
@@
       (effects (font (size 1 1) (thickness 0.15)))
     )
-    (fp_text value IRF1405 (at -4 -8 360) (layer F.SilkS)
-      (effects (font (size 1 1) (thickness 0.15)))
-    )
+    (fp_text value IRFB_7437 (at -3 -8 360) (layer F.SilkS)
+      (effects (font (size 1 1) (thickness 0.15)))
+    )
